File: KiCad/Current Sources Improved.kicad_sch (KiCad schematic)
At the start: 0 parts

Commit message: Cleaned up a few things
Other:
- company: Matt Morano -> M Morano
Changed lines of the file:
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@@
 (kicad_sch (version 20230121) (generator eeschema)
-  (paper "A")
+  (paper "A4")
   (title_block
     (title "Precision Current Source")
     (date "2024-05-20")
     (rev "2.0")
-    (company "Matt Morano")
+    (company "M Morano")
   )
   (junction (at 118.11 78.74) (diameter 0) (color 0 0 0 0)
@@
     (stroke (width 0) (type default))
   )
-  (sheet (at 124.46 88.9) (size 38.1 30.48) (fields_autoplaced)
+  (sheet (at 124.46 88.9) (size 38.735 30.48) (fields_autoplaced)
     (stroke (width 0.1524) (type solid))
     (fill (color 0 0 0 0.0000))
@@
     )
   )
-  (sheet (at 68.58 67.31) (size 43.18 52.07) (fields_autoplaced)
+  (sheet (at 88.9 67.31) (size 22.86 52.07) (fields_autoplaced)
     (stroke (width 0.1524) (type solid))
     (fill (color 0 0 0 0.0000))
-    (property "Sheetname" "Analog" (at 68.58 66.5984 0)
+    (property "Sheetname" "Analog" (at 88.9 66.5984 0)
       (effects (font (size 1.27 1.27)) (justify left bottom))
     )
-    (property "Sheetfile" "Analog.kicad_sch" (at 68.58 119.9646 0)
+    (property "Sheetfile" "Analog.kicad_sch" (at 88.9 119.9646 0)
       (effects (font (size 1.27 1.27)) (justify left top))
     )
@@
     )
   )
-  (sheet (at 124.46 67.31) (size 38.1 15.24) (fields_autoplaced)
+  (sheet (at 124.46 67.31) (size 38.735 15.24) (fields_autoplaced)
     (stroke (width 0.1524) (type solid))
     (fill (color 0 0 0 0.0000))
